File: Power section.kicad_sch (KiCad schematic)
At the start: 17 parts, among them J2 USB3_A, U4 TLV76733, U5 USBLC6-2P6, U6 TPS7A0212

Commit message: Datasheets for all the ICs added iin the Docs folder
Parts:
- U6: footprint TPS7A0230PDQNR:IC_TPS7A0230PDQNR -> TPS7A0212:Tps_7a0212
Changed lines of the file:
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@@
 			)
 		)
-		(property "Footprint" "TPS7A0230PDQNR:IC_TPS7A0230PDQNR"
+		(property "Footprint" "TPS7A0212:Tps_7a0212"
 			(at 127 74.93 0)
 			(hide yes)
